Commit message: Added file so the robot can be simulated in gazebo

File: description/robot.urdf.xacro (robot description, xacro)
@@ -2,3 +2,4 @@
 <robot xmlns:xacro = "http://www.ros.org/wiki/xacro"  name = "robot">
     <xacro:include filename = "robot_core.xacro"/>
+    <xacro:include filename = "gazebo_control.xacro"/>
 </robot>

File: description/robot_core.xacro (robot description, xacro)
@@ -37,4 +37,9 @@
         </xacro:inertial_box>
     </link>
+    <gazebo reference = "chassis">
+        <material>
+            Gazebo/Black
+        </material>
+    </gazebo>
     <!-- Chassis/Base Joint -->
     <joint name = "chassis_joint" type = "fixed">
@@ -46,5 +51,5 @@
     <link name = "left_wheel">
         <visual>
-            <origin xyz = "0 0 0.075"/>
+            <origin xyz = "0 0 0"/>
             <geometry>
                 <cylinder radius = "0.05" length = "0.04"/>
@@ -53,5 +58,5 @@
         </visual>
         <collision>
-            <origin xyz = "0 0 0.075"/>
+            <origin xyz = "0 0 0"/>
             <geometry>
                 <cylinder radius = "0.05" length = "0.04"/>
@@ -59,12 +64,17 @@
         </collision>
         <xacro:inertial_cylinder mass = "0.1" length = "0.04" radius = "0.05">
-            <origin xyz = "0 0 0.075" rpy = "0 0 0"/>
+            <origin xyz = "0 0 0" rpy = "0 0 0"/>
         </xacro:inertial_cylinder>
     </link>
+    <gazebo reference = "left_wheel">
+        <material>
+            Gazebo/Orange
+        </material>
+    </gazebo>
     <!-- Left Wheel Joint -->
     <joint name = "left_wheel_joint" type = "continuous">
         <parent link = "base_link"/>
         <child link = "left_wheel"/>
-        <origin xyz = "0 0.095 0" rpy = "-${pi/2} 0 0"/>
+        <origin xyz = "0 0.175 0" rpy = "-${pi/2} 0 0"/>
         <axis xyz = " 0 0 1"/>
     </joint>
@@ -72,5 +82,5 @@
     <link name = "right_wheel">
         <visual>
-            <origin xyz = "0 0 0.075"/>
+            <origin xyz = "0 0 0"/>
             <geometry>
                 <cylinder radius = "0.05" length = "0.04"/>
@@ -79,5 +89,5 @@
         </visual>
         <collision>
-            <origin xyz = "0 0 0.075"/>
+            <origin xyz = "0 0 0"/>
             <geometry>
                 <cylinder radius = "0.05" length = "0.04"/>
@@ -85,12 +95,17 @@
         </collision>
         <xacro:inertial_cylinder mass = "0.1" length = "0.04" radius = "0.05">
-            <origin xyz = "0 0 0.075" rpy = "0 0 0"/>
+            <origin xyz = "0 0 0" rpy = "0 0 0"/>
         </xacro:inertial_cylinder>
     </link>
+    <gazebo reference = "right_wheel">
+        <material>
+            Gazebo/Orange
+        </material>
+    </gazebo>
     <!-- Right Wheel Joint -->
     <joint name = "right_wheel_joint" type = "continuous">
         <parent link = "base_link"/>
         <child link = "right_wheel"/>
-        <origin xyz = "0 -0.095 0" rpy = "${pi/2} 0 0"/>
+        <origin xyz = "0 -0.175 0" rpy = "${pi/2} 0 0"/>
         <axis xyz = " 0 0 -1"/>
     </joint>
@@ -113,4 +128,11 @@
         </xacro:inertial_sphere>
     </link>
+    <gazebo reference = "caster_front">
+        <material>
+            Gazebo/White
+        </material>
+        <mu1 value = "0.001"/>
+        <mu2 value = "0.001"/>
+    </gazebo>
     <!-- Caster Front Wheel Joint -->
     <joint name = "caster_front_wheel" type = "fixed">
@@ -137,4 +159,11 @@
         </xacro:inertial_sphere>
     </link>
+    <gazebo reference = "caster_back">
+        <material>
+            Gazebo/White
+        </material>
+        <mu1 value = "0.001"/>
+        <mu2 value = "0.001"/>
+    </gazebo>
     <!-- Caster Back Wheel Joint -->
     <joint name = "caster_back_wheel" type = "fixed">

Commit message: Added file to simulate lidar

File: description/robot.urdf.xacro (robot description, xacro)
@@ -3,3 +3,4 @@
     <xacro:include filename = "robot_core.xacro"/>
     <xacro:include filename = "gazebo_control.xacro"/>
+    <xacro:include filename = "lidar.xacro"/>
 </robot>

File: description/robot_core.xacro (robot description, xacro)
@@ -14,4 +14,7 @@
     <material name = "blue">
         <color rgba = "0 0 1 1"/>
+    </material>
+    <material name = "red">
+        <color rgba = "1 0 0 1"/>
     </material>
     <!-- Base Link -->

Commit message: Added new file that makes simulation better and modified some files to make it easier to change between ros2_control and gaze control

File: description/robot.urdf.xacro (robot description, xacro)
@@ -1,7 +1,12 @@
 <?xml version = "1.0"?>
 <robot xmlns:xacro = "http://www.ros.org/wiki/xacro"  name = "robot">
+    <xacro:arg name="use_ros2_control" default="true"/>
     <xacro:include filename = "robot_core.xacro"/>
-    <!-- <xacro:include filename = "gazebo_control.xacro"/> -->
-    <xacro:include filename = "ros2_control.xacro"/>
+    <xacro:if value="$(arg use_ros2_control)">
+        <xacro:include filename = "ros2_control.xacro"/>
+    </xacro:if>
+    <xacro:unless value="$(arg use_ros2_control)">
+        <xacro:include filename = "gazebo_control.xacro"/>
+    </xacro:unless>
     <xacro:include filename = "lidar.xacro"/>
     <!-- <xacro:include filename = "camera.xacro"/> -->

File: description/robot_core.xacro (robot description, xacro)
@@ -63,5 +63,5 @@
             <origin xyz = "0 0 0"/>
             <geometry>
-                <cylinder radius = "0.05" length = "0.04"/>
+                <sphere radius = "0.05"/>
             </geometry>
         </collision>
@@ -94,5 +94,5 @@
             <origin xyz = "0 0 0"/>
             <geometry>
-                <cylinder radius = "0.05" length = "0.04"/>
+                <sphere radius = "0.05"/>
             </geometry>
         </collision>

Commit message: Added code to allow for movement for sim and real rover

File: description/robot.urdf.xacro (robot description, xacro)
@@ -2,4 +2,5 @@
 <robot xmlns:xacro = "http://www.ros.org/wiki/xacro"  name = "robot">
     <xacro:arg name="use_ros2_control" default="true"/>
+    <xacro:arg name="sim_mode" default="false"/>
     <xacro:include filename = "robot_core.xacro"/>
     <xacro:if value="$(arg use_ros2_control)">

File: description/ros2_control.xacro (robot description, xacro)
@@ -1,28 +1,61 @@
 <?xml version="1.0"?>
 <robot xmlns:xacro="http://www.ros.org/wiki/xacro">
-    <ros2_control name="GazeboSystem" type="system">
-        <hardware>
-            <plugin>gazebo_ros2_control/GazeboSystem</plugin>
-        </hardware>
-        <joint name="left_wheel_joint">
-            <command_interface name="velocity">
-                <param name="min">-10</param>
-                <param name="max">10</param>
-            </command_interface>
-            <state_interface name="velocity"/>
-            <state_interface name="position"/>
-        </joint>
-        <joint name="right_wheel_joint">
-            <command_interface name="velocity">
-                <param name="min">-10</param>
-                <param name="max">10</param>
-            </command_interface>
-            <state_interface name="velocity"/>
-            <state_interface name="position"/>
-        </joint>
-    </ros2_control>
+    <xacro:if value="$(arg sim_mode)">
+        <ros2_control name="GazeboSystem" type="system">
+            <hardware>
+                <plugin>gazebo_ros2_control/GazeboSystem</plugin>
+            </hardware>
+            <joint name="left_wheel_joint">
+                <command_interface name="velocity">
+                    <param name="min">-10</param>
+                    <param name="max">10</param>
+                </command_interface>
+                <state_interface name="velocity"/>
+                <state_interface name="position"/>
+            </joint>
+            <joint name="right_wheel_joint">
+                <command_interface name="velocity">
+                    <param name="min">-10</param>
+                    <param name="max">10</param>
+                </command_interface>
+                <state_interface name="velocity"/>
+                <state_interface name="position"/>
+            </joint>
+        </ros2_control>
+    </xacro:if>
+    <xacro:unless value="$(arg sim_mode)">
+        <ros2_control name="RealRobot" type="system">
+            <hardware>
+                <plugin>diffdrive_arduino/DiffDriveArduino</plugin>
+                <param name="left_wheel_name">left_wheel_joint</param>
+                <param name="right_wheel_name">right_wheel_joint</param>
+                <param name="loop_rate">30</param>
+                <param name="device">/dev/ttyUSB0</param>
+                <param name="baud_rate">57600</param>
+                <param name="timeout">1000</param>
+                <param name="enc_counts_per_rev">3436</param>
+            </hardware>
+            <joint name="left_wheel_joint">
+                <command_interface name="velocity">
+                    <param name="min">-10</param>
+                    <param name="max">10</param>
+                </command_interface>
+                <state_interface name="velocity"/>
+                <state_interface name="position"/>
+            </joint>
+            <joint name="right_wheel_joint">
+                <command_interface name="velocity">
+                    <param name="min">-10</param>
+                    <param name="max">10</param>
+                </command_interface>
+                <state_interface name="velocity"/>
+                <state_interface name="position"/>
+            </joint>
+        </ros2_control>
+    </xacro:unless>
     <gazebo>
         <plugin name="gazebo_ros2_control" filename="libgazebo_ros2_control.so">
             <parameters>$(find Theseus)/config/my_controllers.yaml</parameters>
+            <parameters>$(find Theseus)/config/gaz_ros2_ctl_use_sim.yaml</parameters>
         </plugin>
     </gazebo>
