Commit message: Added SLAM and Automation files

File: description/robot_core.xacro (robot description, xacro)
@@ -21,4 +21,13 @@
     <link name = "base_link">
     </link>
+    <!-- Base Footprint Link -->
+    <link name="base_footprint">
+    </link>
+    <!-- Base Footprint Joint -->
+    <joint name="base_foorprint_joint" type="fixed">
+        <parent link="base_link"/>
+        <child link="base_footprint"/>
+        <origin xyz="0 0 0" rpy="0 0 0"/>
+    </joint>
     <!-- Chassis Link -->
     <link name = "chassis">

Commit message: Adding changes to actual rover

File: description/robot_core.xacro (robot description, xacro)
@@ -122,10 +122,10 @@
         <axis xyz = " 0 0 -1"/>
     </joint>
-    <!-- Caster Front Wheel Link -->
-    <link name = "caster_front">
+    <!-- Caster Back Wheel Link -->
+    <link name = "caster_back">
         <visual>
             <origin xyz = "0 0 0"/>
             <geometry>
-                <sphere radius = "0.015"/>
+                <sphere radius = "0.025"/>
             </geometry>
             <material name = "white"/>
@@ -133,12 +133,12 @@
         <collision>
             <geometry>
-                <sphere radius = "0.015"/>
+                <sphere radius = "0.025"/>
             </geometry>
         </collision>
-        <xacro:inertial_sphere mass = "0.1" radius = "0.015">
+        <xacro:inertial_sphere mass = "0.1" radius = "0.025">
             <origin xyz = "0 0 0" rpy = "0 0 0"/>
         </xacro:inertial_sphere>
     </link>
-    <gazebo reference = "caster_front">
+    <gazebo reference = "caster_back">
         <material>
             Gazebo/White
@@ -147,9 +147,9 @@
         <mu2 value = "0.001"/>
     </gazebo>
-    <!-- Caster Front Wheel Joint -->
-    <joint name = "caster_front_wheel" type = "fixed">
+    <!-- Caster Back Wheel Joint -->
+    <joint name = "caster_back_wheel" type = "fixed">
         <parent link = "chassis"/>
-        <child link = "caster_front"/>
-        <origin xyz = "-0.022 0 -0.01"/>
+        <child link = "caster_back"/>
+        <origin xyz = "-0.022 0 -0.009"/>
     </joint>
 </robot>
