Commit message: Changing wheel radius

File: description/robot_core.xacro (robot description, xacro)
@@ -65,5 +65,5 @@
             <origin xyz = "0 0 0"/>
             <geometry>
-                <cylinder radius = "0.03375" length = "0.026"/>
+                <cylinder radius = "0.09704" length = "0.026"/>
             </geometry>
             <material name = "orange"/>
@@ -72,8 +72,8 @@
             <origin xyz = "0 0 0"/>
             <geometry>
-                <sphere radius = "0.03375"/>
+                <sphere radius = "0.09704"/>
             </geometry>
         </collision>
-        <xacro:inertial_cylinder mass = "0.1" length = "0.026" radius = "0.03375">
+        <xacro:inertial_cylinder mass = "0.1" length = "0.026" radius = "0.09704">
             <origin xyz = "0 0 0" rpy = "0 0 0"/>
         </xacro:inertial_cylinder>
@@ -96,5 +96,5 @@
             <origin xyz = "0 0 0"/>
             <geometry>
-                <cylinder radius = "0.03375" length = "0.026"/>
+                <cylinder radius = "0.09704" length = "0.026"/>
             </geometry>
             <material name = "orange"/>
@@ -103,8 +103,8 @@
             <origin xyz = "0 0 0"/>
             <geometry>
-                <sphere radius = "0.03375"/>
+                <sphere radius = "0.09704"/>
             </geometry>
         </collision>
-        <xacro:inertial_cylinder mass = "0.1" length = "0.026" radius = "0.03375">
+        <xacro:inertial_cylinder mass = "0.1" length = "0.026" radius = "0.09704">
             <origin xyz = "0 0 0" rpy = "0 0 0"/>
         </xacro:inertial_cylinder>
@@ -127,5 +127,5 @@
             <origin xyz = "0 0 0"/>
             <geometry>
-                <sphere radius = "0.025"/>
+                <sphere radius = "0.09704"/>
             </geometry>
             <material name = "white"/>
@@ -133,8 +133,8 @@
         <collision>
             <geometry>
-                <sphere radius = "0.025"/>
+                <sphere radius = "0.09704"/>
             </geometry>
         </collision>
-        <xacro:inertial_sphere mass = "0.1" radius = "0.025">
+        <xacro:inertial_sphere mass = "0.1" radius = "0.09704">
             <origin xyz = "0 0 0" rpy = "0 0 0"/>
         </xacro:inertial_sphere>
@@ -158,5 +158,5 @@
             <origin xyz = "0 0 0"/>
             <geometry>
-                <sphere radius = "0.025"/>
+                <sphere radius = "0.09704"/>
             </geometry>
             <material name = "white"/>
@@ -164,8 +164,8 @@
         <collision>
             <geometry>
-                <sphere radius = "0.025"/>
+                <sphere radius = "0.09704"/>
             </geometry>
         </collision>
-        <xacro:inertial_sphere mass = "0.1" radius = "0.025">
+        <xacro:inertial_sphere mass = "0.1" radius = "0.09704">
             <origin xyz = "0 0 0" rpy = "0 0 0"/>
         </xacro:inertial_sphere>

Commit message: Added files to make robot sim better and controller use

File: description/robot_core.xacro (robot description, xacro)
@@ -127,5 +127,5 @@
             <origin xyz = "0 0 0"/>
             <geometry>
-                <sphere radius = "0.09704"/>
+                <sphere radius = "0.025"/>
             </geometry>
             <material name = "white"/>
@@ -133,8 +133,8 @@
         <collision>
             <geometry>
-                <sphere radius = "0.09704"/>
+                <sphere radius = "0.025"/>
             </geometry>
         </collision>
-        <xacro:inertial_sphere mass = "0.1" radius = "0.09704">
+        <xacro:inertial_sphere mass = "0.1" radius = "0.025">
             <origin xyz = "0 0 0" rpy = "0 0 0"/>
         </xacro:inertial_sphere>
@@ -151,5 +151,5 @@
         <parent link = "chassis"/>
         <child link = "caster_back"/>
-        <origin xyz = "0.025 0 -0.009"/>
+        <origin xyz = "0.025 0 -0.07204"/>
     </joint>
     <!-- Caster Front Wheel Link -->
@@ -158,5 +158,5 @@
             <origin xyz = "0 0 0"/>
             <geometry>
-                <sphere radius = "0.09704"/>
+                <sphere radius = "0.025"/>
             </geometry>
             <material name = "white"/>
@@ -164,8 +164,8 @@
         <collision>
             <geometry>
-                <sphere radius = "0.09704"/>
+                <sphere radius = "0.025"/>
             </geometry>
         </collision>
-        <xacro:inertial_sphere mass = "0.1" radius = "0.09704">
+        <xacro:inertial_sphere mass = "0.1" radius = "0.025">
             <origin xyz = "0 0 0" rpy = "0 0 0"/>
         </xacro:inertial_sphere>
@@ -182,5 +182,5 @@
         <parent link = "chassis"/>
         <child link = "caster_front"/>
-        <origin xyz = "0.225 0 -0.009"/>
+        <origin xyz = "0.225 0 -0.07204"/>
     </joint>
 </robot>
