Commit message: Made changes to reflect actual rover

File: description/camera.xacro (robot description, xacro)
@@ -6,5 +6,5 @@
             <origin xyz = "0 0 0" rpy = "0 0 0"/>
             <geometry>
-                <box size = "0.010 0.03 0.03"/>
+                <box size = "0.020 0.072 0.032"/>
             </geometry>
             <material name = "red"/>
@@ -40,5 +40,5 @@
         <parent link = "chassis"/>
         <child link = "camera_link"/>
-        <origin xyz = "0.305 0 0.08" rpy = "0 0 0"/>
+        <origin xyz = "0.201 0 0.075" rpy = "0 0 0"/>
     </joint>
     <!-- Camera Optical Link -->

File: description/gazebo_control.xacro (robot description, xacro)
@@ -6,6 +6,6 @@
             <left_joint>left_wheel_joint</left_joint>
             <right_joint>right_wheel_joint</right_joint>
-            <wheel_separation>0.35</wheel_separation>
-            <wheel_diameter>0.1</wheel_diameter>
+            <wheel_separation>0.18</wheel_separation>
+            <wheel_diameter>0.134</wheel_diameter>
             <!-- Limits -->
             <max_wheel_torque>200</max_wheel_torque>

File: description/lidar.xacro (robot description, xacro)
@@ -6,5 +6,5 @@
             <origin xyz = "0 0 0" rpy = "0 0 0"/>
             <geometry>
-                <cylinder radius = "0.05" length = "0.04"/>
+                <cylinder radius = "0.038" length = "0.04"/>
             </geometry>
             <material name = "red"/>
@@ -13,8 +13,8 @@
             <origin xyz = "0 0 0" rpy = "0 0 0"/>
             <geometry>
-                <cylinder radius = "0.05" length = "0.04"/>
+                <cylinder radius = "0.038" length = "0.04"/>
             </geometry>
         </collision>
-        <xacro:inertial_cylinder mass = "0.1" length = "0.04" radius = "0.05">
+        <xacro:inertial_cylinder mass = "0.1" length = "0.04" radius = "0.038">
             <origin xyz = "0 0 0" rpy = "0 0 0"/>
         </xacro:inertial_cylinder>
@@ -54,5 +54,5 @@
         <parent link = "chassis"/>
         <child link = "laser_frame"/>
-        <origin xyz = "0.1 0 0.175" rpy = "0 0 0"/>
+        <origin xyz = "0.07 0 0.13" rpy = "0 0 0"/>
     </joint>
 </robot>

File: description/robot_core.xacro (robot description, xacro)
@@ -33,18 +33,18 @@
     <link name = "chassis">
         <visual>
-            <origin xyz = "0.15 0 0.075"/>
+            <origin xyz = "0.07 0 0.05"/>
             <geometry>
-                <box size = ".3 .3 .15"/>
+                <box size = "0.245 0.15 0.123"/>
             </geometry>
             <material name = "black"/>
         </visual>
         <collision>
-            <origin xyz = "0.15 0 0.075"/>
+            <origin xyz = "0.07 0 0.05"/>
             <geometry>
-                <box size = ".3 .3 .15"/>
+                <box size = "0.245 0.15 0.123"/>
             </geometry>
         </collision>
-        <xacro:inertial_box mass = "0.5" x = "0.3" y = "0.3" z = "0.15">
-            <origin xyz = "0.15 0 0.075" rpy = "0 0 0"/>
+        <xacro:inertial_box mass = "0.5" x = "0.245" y = "0.15" z = "0.123">
+            <origin xyz = "0.07 0 0.05" rpy = "0 0 0"/>
         </xacro:inertial_box>
     </link>
@@ -65,5 +65,5 @@
             <origin xyz = "0 0 0"/>
             <geometry>
-                <cylinder radius = "0.05" length = "0.04"/>
+                <cylinder radius = "0.033" length = "0.025"/>
             </geometry>
             <material name = "orange"/>
@@ -72,8 +72,8 @@
             <origin xyz = "0 0 0"/>
             <geometry>
-                <sphere radius = "0.05"/>
+                <sphere radius = "0.033"/>
             </geometry>
         </collision>
-        <xacro:inertial_cylinder mass = "0.1" length = "0.04" radius = "0.05">
+        <xacro:inertial_cylinder mass = "0.1" length = "0.025" radius = "0.033">
             <origin xyz = "0 0 0" rpy = "0 0 0"/>
         </xacro:inertial_cylinder>
@@ -88,5 +88,5 @@
         <parent link = "base_link"/>
         <child link = "left_wheel"/>
-        <origin xyz = "0 0.175 0" rpy = "-${pi/2} 0 0"/>
+        <origin xyz = "0 0.09 0" rpy = "-${pi/2} 0 0"/>
         <axis xyz = " 0 0 1"/>
     </joint>
@@ -96,5 +96,5 @@
             <origin xyz = "0 0 0"/>
             <geometry>
-                <cylinder radius = "0.05" length = "0.04"/>
+                <cylinder radius = "0.033" length = "0.025"/>
             </geometry>
             <material name = "orange"/>
@@ -103,8 +103,8 @@
             <origin xyz = "0 0 0"/>
             <geometry>
-                <sphere radius = "0.05"/>
+                <sphere radius = "0.033"/>
             </geometry>
         </collision>
-        <xacro:inertial_cylinder mass = "0.1" length = "0.04" radius = "0.05">
+        <xacro:inertial_cylinder mass = "0.1" length = "0.025" radius = "0.033">
             <origin xyz = "0 0 0" rpy = "0 0 0"/>
         </xacro:inertial_cylinder>
@@ -119,5 +119,5 @@
         <parent link = "base_link"/>
         <child link = "right_wheel"/>
-        <origin xyz = "0 -0.175 0" rpy = "${pi/2} 0 0"/>
+        <origin xyz = "0 -0.09 0" rpy = "${pi/2} 0 0"/>
         <axis xyz = " 0 0 -1"/>
     </joint>
@@ -127,5 +127,5 @@
             <origin xyz = "0 0 0"/>
             <geometry>
-                <sphere radius = "0.05"/>
+                <sphere radius = "0.015"/>
             </geometry>
             <material name = "white"/>
@@ -133,8 +133,8 @@
         <collision>
             <geometry>
-                <sphere radius = "0.05"/>
+                <sphere radius = "0.015"/>
             </geometry>
         </collision>
-        <xacro:inertial_sphere mass = "0.1" radius = "0.05">
+        <xacro:inertial_sphere mass = "0.1" radius = "0.015">
             <origin xyz = "0 0 0" rpy = "0 0 0"/>
         </xacro:inertial_sphere>
@@ -151,36 +151,5 @@
         <parent link = "chassis"/>
         <child link = "caster_front"/>
-        <origin xyz = "0.25 0 0"/>
-    </joint>
-    <!-- Caster Back Wheel Link -->
-    <link name = "caster_back">
-        <visual>
-            <origin xyz = "0 0 0"/>
-            <geometry>
-                <sphere radius = "0.05"/>
-            </geometry>
-            <material name = "white"/>
-        </visual>
-        <collision>
-            <geometry>
-                <sphere radius = "0.05"/>
-            </geometry>
-        </collision>
-        <xacro:inertial_sphere mass = "0.1" radius = "0.05">
-            <origin xyz = "0 0 0" rpy = "0 0 0"/>
-        </xacro:inertial_sphere>
-    </link>
-    <gazebo reference = "caster_back">
-        <material>
-            Gazebo/White
-        </material>
-        <mu1 value = "0.001"/>
-        <mu2 value = "0.001"/>
-    </gazebo>
-    <!-- Caster Back Wheel Joint -->
-    <joint name = "caster_back_wheel" type = "fixed">
-        <parent link = "chassis"/>
-        <child link = "caster_back"/>
-        <origin xyz = "0.05 0 0"/>
+        <origin xyz = "-0.022 0 -0.01"/>
     </joint>
 </robot>

Commit message: Changed certains things to get things closer to real life rover

File: description/camera.xacro (robot description, xacro)
@@ -40,5 +40,5 @@
         <parent link = "chassis"/>
         <child link = "camera_link"/>
-        <origin xyz = "0.201 0 0.075" rpy = "0 0 0"/>
+        <origin xyz = "0.240 0 0.080" rpy = "0 0 0"/>
     </joint>
     <!-- Camera Optical Link -->

File: description/gazebo_control.xacro (robot description, xacro)
@@ -7,5 +7,5 @@
             <right_joint>right_wheel_joint</right_joint>
             <wheel_separation>0.18</wheel_separation>
-            <wheel_diameter>0.134</wheel_diameter>
+            <wheel_diameter>0.0675</wheel_diameter>
             <!-- Limits -->
             <max_wheel_torque>200</max_wheel_torque>

File: description/lidar.xacro (robot description, xacro)
@@ -54,5 +54,5 @@
         <parent link = "chassis"/>
         <child link = "laser_frame"/>
-        <origin xyz = "0.07 0 0.13" rpy = "0 0 0"/>
+        <origin xyz = "0.1 0 0.123" rpy = "0 0 0"/>
     </joint>
 </robot>

File: description/robot_core.xacro (robot description, xacro)
@@ -33,5 +33,5 @@
     <link name = "chassis">
         <visual>
-            <origin xyz = "0.07 0 0.05"/>
+            <origin xyz = "0.11 0 0.0415"/>
             <geometry>
                 <box size = "0.245 0.15 0.123"/>
@@ -40,5 +40,5 @@
         </visual>
         <collision>
-            <origin xyz = "0.07 0 0.05"/>
+            <origin xyz = "0.11 0 0.0415"/>
             <geometry>
                 <box size = "0.245 0.15 0.123"/>
@@ -46,5 +46,5 @@
         </collision>
         <xacro:inertial_box mass = "0.5" x = "0.245" y = "0.15" z = "0.123">
-            <origin xyz = "0.07 0 0.05" rpy = "0 0 0"/>
+            <origin xyz = "0.11 0 0.0415" rpy = "0 0 0"/>
         </xacro:inertial_box>
     </link>
@@ -58,5 +58,5 @@
         <parent link = "base_link"/>
         <child link = "chassis"/>
-        <origin xyz = "-0.15 0 0"/>
+        <origin xyz = "-0.210 0 0"/>
     </joint>
     <!-- Left Wheel Link -->
@@ -65,5 +65,5 @@
             <origin xyz = "0 0 0"/>
             <geometry>
-                <cylinder radius = "0.033" length = "0.025"/>
+                <cylinder radius = "0.03375" length = "0.026"/>
             </geometry>
             <material name = "orange"/>
@@ -72,8 +72,8 @@
             <origin xyz = "0 0 0"/>
             <geometry>
-                <sphere radius = "0.033"/>
+                <sphere radius = "0.03375"/>
             </geometry>
         </collision>
-        <xacro:inertial_cylinder mass = "0.1" length = "0.025" radius = "0.033">
+        <xacro:inertial_cylinder mass = "0.1" length = "0.026" radius = "0.03375">
             <origin xyz = "0 0 0" rpy = "0 0 0"/>
         </xacro:inertial_cylinder>
@@ -96,5 +96,5 @@
             <origin xyz = "0 0 0"/>
             <geometry>
-                <cylinder radius = "0.033" length = "0.025"/>
+                <cylinder radius = "0.03375" length = "0.026"/>
             </geometry>
             <material name = "orange"/>
@@ -103,8 +103,8 @@
             <origin xyz = "0 0 0"/>
             <geometry>
-                <sphere radius = "0.033"/>
+                <sphere radius = "0.03375"/>
             </geometry>
         </collision>
-        <xacro:inertial_cylinder mass = "0.1" length = "0.025" radius = "0.033">
+        <xacro:inertial_cylinder mass = "0.1" length = "0.026" radius = "0.03375">
             <origin xyz = "0 0 0" rpy = "0 0 0"/>
         </xacro:inertial_cylinder>
@@ -151,5 +151,5 @@
         <parent link = "chassis"/>
         <child link = "caster_back"/>
-        <origin xyz = "-0.022 0 -0.009"/>
+        <origin xyz = "0.025 0 -0.009"/>
     </joint>
 </robot>
