Commit message: Change simulation details

File: description/camera.xacro (robot description, xacro)
@@ -40,5 +40,5 @@
         <parent link = "chassis"/>
         <child link = "camera_link"/>
-        <origin xyz = "0.240 0 0.080" rpy = "0 0 0"/>
+        <origin xyz = "0.260 0 0.080" rpy = "0 0 0"/>
     </joint>
     <!-- Camera Optical Link -->

File: description/lidar.xacro (robot description, xacro)
@@ -54,5 +54,5 @@
         <parent link = "chassis"/>
         <child link = "laser_frame"/>
-        <origin xyz = "0.11 0 0.123" rpy = "0 0 0"/>
+        <origin xyz = "0.125 0 0.123" rpy = "0 0 0"/>
     </joint>
 </robot>

File: description/robot_core.xacro (robot description, xacro)
@@ -33,18 +33,18 @@
     <link name = "chassis">
         <visual>
-            <origin xyz = "0.11 0 0.0415"/>
+            <origin xyz = "0.125 0 0.0415"/>
             <geometry>
-                <box size = "0.245 0.15 0.123"/>
+                <box size = "0.250 0.155 0.123"/>
             </geometry>
             <material name = "black"/>
         </visual>
         <collision>
-            <origin xyz = "0.11 0 0.0415"/>
+            <origin xyz = "0.125 0 0.0415"/>
             <geometry>
-                <box size = "0.245 0.15 0.123"/>
+                <box size = "0.250 0.155 0.123"/>
             </geometry>
         </collision>
-        <xacro:inertial_box mass = "0.5" x = "0.245" y = "0.15" z = "0.123">
-            <origin xyz = "0.11 0 0.0415" rpy = "0 0 0"/>
+        <xacro:inertial_box mass = "0.5" x = "0.250" y = "0.155" z = "0.123">
+            <origin xyz = "0.125 0 0.0415" rpy = "0 0 0"/>
         </xacro:inertial_box>
     </link>
@@ -58,5 +58,5 @@
         <parent link = "base_link"/>
         <child link = "chassis"/>
-        <origin xyz = "-0.210 0 0"/>
+        <origin xyz = "-0.125 0 0"/>
     </joint>
     <!-- Left Wheel Link -->
@@ -151,5 +151,36 @@
         <parent link = "chassis"/>
         <child link = "caster_back"/>
-        <origin xyz = "0.0155 0 -0.009"/>
+        <origin xyz = "0.025 0 -0.009"/>
+    </joint>
+    <!-- Caster Front Wheel Link -->
+    <link name = "caster_front">
+        <visual>
+            <origin xyz = "0 0 0"/>
+            <geometry>
+                <sphere radius = "0.025"/>
+            </geometry>
+            <material name = "white"/>
+        </visual>
+        <collision>
+            <geometry>
+                <sphere radius = "0.025"/>
+            </geometry>
+        </collision>
+        <xacro:inertial_sphere mass = "0.1" radius = "0.025">
+            <origin xyz = "0 0 0" rpy = "0 0 0"/>
+        </xacro:inertial_sphere>
+    </link>
+    <gazebo reference = "caster_front">
+        <material>
+            Gazebo/White
+        </material>
+        <mu1 value = "0.001"/>
+        <mu2 value = "0.001"/>
+    </gazebo>
+    <!-- Caster Front Wheel Joint -->
+    <joint name = "caster_front_wheel" type = "fixed">
+        <parent link = "chassis"/>
+        <child link = "caster_front"/>
+        <origin xyz = "0.225 0 -0.009"/>
     </joint>
 </robot>
