Commit message: Moving lidar and slowing down rover

File: description/lidar.xacro (robot description, xacro)
@@ -54,5 +54,5 @@
         <parent link = "chassis"/>
         <child link = "laser_frame"/>
-        <origin xyz = "0.1 0 0.123" rpy = "0 0 0"/>
+        <origin xyz = "0.11 0 0.123" rpy = "0 0 0"/>
     </joint>
 </robot>

File: description/ros2_control.xacro (robot description, xacro)
@@ -8,6 +8,6 @@
             <joint name="left_wheel_joint">
                 <command_interface name="velocity">
-                    <param name="min">-5</param>
-                    <param name="max">5</param>
+                    <param name="min">-2</param>
+                    <param name="max">2</param>
                 </command_interface>
                 <state_interface name="velocity"/>
@@ -16,6 +16,6 @@
             <joint name="right_wheel_joint">
                 <command_interface name="velocity">
-                    <param name="min">-5</param>
-                    <param name="max">5</param>
+                    <param name="min">-2</param>
+                    <param name="max">2</param>
                 </command_interface>
                 <state_interface name="velocity"/>
@@ -38,6 +38,6 @@
             <joint name="left_wheel_joint">
                 <command_interface name="velocity">
-                    <param name="min">-5</param>
-                    <param name="max">5</param>
+                    <param name="min">-2</param>
+                    <param name="max">2</param>
                 </command_interface>
                 <state_interface name="velocity"/>
@@ -46,6 +46,6 @@
             <joint name="right_wheel_joint">
                 <command_interface name="velocity">
-                    <param name="min">-5</param>
-                    <param name="max">5</param>
+                    <param name="min">-2</param>
+                    <param name="max">2</param>
                 </command_interface>
                 <state_interface name="velocity"/>
