Commit message: Changing tire numbers

File: description/gazebo_control.xacro (robot description, xacro)
@@ -6,5 +6,5 @@
             <left_joint>left_wheel_joint</left_joint>
             <right_joint>right_wheel_joint</right_joint>
-            <wheel_separation>0.18</wheel_separation>
+            <wheel_separation>0.192</wheel_separation>
             <wheel_diameter>0.0675</wheel_diameter>
             <!-- Limits -->

File: description/robot_core.xacro (robot description, xacro)
@@ -88,5 +88,5 @@
         <parent link = "base_link"/>
         <child link = "left_wheel"/>
-        <origin xyz = "0 0.09 0" rpy = "-${pi/2} 0 0"/>
+        <origin xyz = "0 0.096 0" rpy = "-${pi/2} 0 0"/>
         <axis xyz = " 0 0 1"/>
     </joint>
@@ -119,5 +119,5 @@
         <parent link = "base_link"/>
         <child link = "right_wheel"/>
-        <origin xyz = "0 -0.09 0" rpy = "${pi/2} 0 0"/>
+        <origin xyz = "0 -0.096 0" rpy = "${pi/2} 0 0"/>
         <axis xyz = " 0 0 -1"/>
     </joint>

Commit message: Changing tire numbers

File: description/gazebo_control.xacro (robot description, xacro)
@@ -6,5 +6,5 @@
             <left_joint>left_wheel_joint</left_joint>
             <right_joint>right_wheel_joint</right_joint>
-            <wheel_separation>0.192</wheel_separation>
+            <wheel_separation>0.195</wheel_separation>
             <wheel_diameter>0.0675</wheel_diameter>
             <!-- Limits -->

File: description/robot_core.xacro (robot description, xacro)
@@ -88,5 +88,5 @@
         <parent link = "base_link"/>
         <child link = "left_wheel"/>
-        <origin xyz = "0 0.096 0" rpy = "-${pi/2} 0 0"/>
+        <origin xyz = "0 0.0975 0" rpy = "-${pi/2} 0 0"/>
         <axis xyz = " 0 0 1"/>
     </joint>
@@ -119,5 +119,5 @@
         <parent link = "base_link"/>
         <child link = "right_wheel"/>
-        <origin xyz = "0 -0.096 0" rpy = "${pi/2} 0 0"/>
+        <origin xyz = "0 -0.0975 0" rpy = "${pi/2} 0 0"/>
         <axis xyz = " 0 0 -1"/>
     </joint>

Commit message: Changing tire numbers

File: description/gazebo_control.xacro (robot description, xacro)
@@ -6,5 +6,5 @@
             <left_joint>left_wheel_joint</left_joint>
             <right_joint>right_wheel_joint</right_joint>
-            <wheel_separation>0.195</wheel_separation>
+            <wheel_separation>0.2</wheel_separation>
             <wheel_diameter>0.0675</wheel_diameter>
             <!-- Limits -->

File: description/robot_core.xacro (robot description, xacro)
@@ -88,5 +88,5 @@
         <parent link = "base_link"/>
         <child link = "left_wheel"/>
-        <origin xyz = "0 0.0975 0" rpy = "-${pi/2} 0 0"/>
+        <origin xyz = "0 0.1 0" rpy = "-${pi/2} 0 0"/>
         <axis xyz = " 0 0 1"/>
     </joint>
@@ -119,5 +119,5 @@
         <parent link = "base_link"/>
         <child link = "right_wheel"/>
-        <origin xyz = "0 -0.0975 0" rpy = "${pi/2} 0 0"/>
+        <origin xyz = "0 -0.1 0" rpy = "${pi/2} 0 0"/>
         <axis xyz = " 0 0 -1"/>
     </joint>

Commit message: Making measurements more accurate

File: description/gazebo_control.xacro (robot description, xacro)
@@ -6,5 +6,5 @@
             <left_joint>left_wheel_joint</left_joint>
             <right_joint>right_wheel_joint</right_joint>
-            <wheel_separation>0.2</wheel_separation>
+            <wheel_separation>0.21</wheel_separation>
             <wheel_diameter>0.0675</wheel_diameter>
             <!-- Limits -->

File: description/robot_core.xacro (robot description, xacro)
@@ -88,5 +88,5 @@
         <parent link = "base_link"/>
         <child link = "left_wheel"/>
-        <origin xyz = "0 0.1 0" rpy = "-${pi/2} 0 0"/>
+        <origin xyz = "0 0.105 0" rpy = "-${pi/2} 0 0"/>
         <axis xyz = " 0 0 1"/>
     </joint>
@@ -119,5 +119,5 @@
         <parent link = "base_link"/>
         <child link = "right_wheel"/>
-        <origin xyz = "0 -0.1 0" rpy = "${pi/2} 0 0"/>
+        <origin xyz = "0 -0.105 0" rpy = "${pi/2} 0 0"/>
         <axis xyz = " 0 0 -1"/>
     </joint>
@@ -151,5 +151,5 @@
         <parent link = "chassis"/>
         <child link = "caster_back"/>
-        <origin xyz = "0.025 0 -0.009"/>
+        <origin xyz = "0.0155 0 -0.009"/>
     </joint>
 </robot>

Commit message: Once again, trying to get numbers right

File: description/gazebo_control.xacro (robot description, xacro)
@@ -6,5 +6,5 @@
             <left_joint>left_wheel_joint</left_joint>
             <right_joint>right_wheel_joint</right_joint>
-            <wheel_separation>0.21</wheel_separation>
+            <wheel_separation>0.2</wheel_separation>
             <wheel_diameter>0.0675</wheel_diameter>
             <!-- Limits -->

File: description/robot_core.xacro (robot description, xacro)
@@ -88,5 +88,5 @@
         <parent link = "base_link"/>
         <child link = "left_wheel"/>
-        <origin xyz = "0 0.105 0" rpy = "-${pi/2} 0 0"/>
+        <origin xyz = "0 0.1 0" rpy = "-${pi/2} 0 0"/>
         <axis xyz = " 0 0 1"/>
     </joint>
@@ -119,5 +119,5 @@
         <parent link = "base_link"/>
         <child link = "right_wheel"/>
-        <origin xyz = "0 -0.105 0" rpy = "${pi/2} 0 0"/>
+        <origin xyz = "0 -0.1 0" rpy = "${pi/2} 0 0"/>
         <axis xyz = " 0 0 -1"/>
     </joint>

Commit message: Parameter change again

File: description/gazebo_control.xacro (robot description, xacro)
@@ -6,5 +6,5 @@
             <left_joint>left_wheel_joint</left_joint>
             <right_joint>right_wheel_joint</right_joint>
-            <wheel_separation>0.2</wheel_separation>
+            <wheel_separation>0.205</wheel_separation>
             <wheel_diameter>0.0675</wheel_diameter>
             <!-- Limits -->

File: description/robot_core.xacro (robot description, xacro)
@@ -88,5 +88,5 @@
         <parent link = "base_link"/>
         <child link = "left_wheel"/>
-        <origin xyz = "0 0.1 0" rpy = "-${pi/2} 0 0"/>
+        <origin xyz = "0 0.1025 0" rpy = "-${pi/2} 0 0"/>
         <axis xyz = " 0 0 1"/>
     </joint>
@@ -119,5 +119,5 @@
         <parent link = "base_link"/>
         <child link = "right_wheel"/>
-        <origin xyz = "0 -0.1 0" rpy = "${pi/2} 0 0"/>
+        <origin xyz = "0 -0.1025 0" rpy = "${pi/2} 0 0"/>
         <axis xyz = " 0 0 -1"/>
     </joint>

Commit message: Parameter change again

File: description/gazebo_control.xacro (robot description, xacro)
@@ -6,5 +6,5 @@
             <left_joint>left_wheel_joint</left_joint>
             <right_joint>right_wheel_joint</right_joint>
-            <wheel_separation>0.205</wheel_separation>
+            <wheel_separation>0.202</wheel_separation>
             <wheel_diameter>0.0675</wheel_diameter>
             <!-- Limits -->

File: description/robot_core.xacro (robot description, xacro)
@@ -88,5 +88,5 @@
         <parent link = "base_link"/>
         <child link = "left_wheel"/>
-        <origin xyz = "0 0.1025 0" rpy = "-${pi/2} 0 0"/>
+        <origin xyz = "0 0.101 0" rpy = "-${pi/2} 0 0"/>
         <axis xyz = " 0 0 1"/>
     </joint>
@@ -119,5 +119,5 @@
         <parent link = "base_link"/>
         <child link = "right_wheel"/>
-        <origin xyz = "0 -0.1025 0" rpy = "${pi/2} 0 0"/>
+        <origin xyz = "0 -0.101 0" rpy = "${pi/2} 0 0"/>
         <axis xyz = " 0 0 -1"/>
     </joint>
