Commit message: Changing to match tank

File: description/gazebo_control.xacro (robot description, xacro)
@@ -6,6 +6,6 @@
             <left_joint>left_wheel_joint</left_joint>
             <right_joint>right_wheel_joint</right_joint>
-            <wheel_separation>0.202</wheel_separation>
-            <wheel_diameter>0.0675</wheel_diameter>
+            <wheel_separation>0.260</wheel_separation>
+            <wheel_diameter>0.09704</wheel_diameter>
             <!-- Limits -->
             <max_wheel_torque>200</max_wheel_torque>

File: description/robot_core.xacro (robot description, xacro)
@@ -65,5 +65,5 @@
             <origin xyz = "0 0 0"/>
             <geometry>
-                <cylinder radius = "0.09704" length = "0.026"/>
+                <cylinder radius = "0.09704" length = "0.041"/>
             </geometry>
             <material name = "orange"/>
@@ -75,5 +75,5 @@
             </geometry>
         </collision>
-        <xacro:inertial_cylinder mass = "0.1" length = "0.026" radius = "0.09704">
+        <xacro:inertial_cylinder mass = "0.1" length = "0.041" radius = "0.09704">
             <origin xyz = "0 0 0" rpy = "0 0 0"/>
         </xacro:inertial_cylinder>
@@ -88,5 +88,5 @@
         <parent link = "base_link"/>
         <child link = "left_wheel"/>
-        <origin xyz = "0 0.101 0" rpy = "-${pi/2} 0 0"/>
+        <origin xyz = "0 0.110 0" rpy = "-${pi/2} 0 0"/>
         <axis xyz = " 0 0 1"/>
     </joint>
@@ -96,5 +96,5 @@
             <origin xyz = "0 0 0"/>
             <geometry>
-                <cylinder radius = "0.09704" length = "0.026"/>
+                <cylinder radius = "0.09704" length = "0.041"/>
             </geometry>
             <material name = "orange"/>
@@ -106,5 +106,5 @@
             </geometry>
         </collision>
-        <xacro:inertial_cylinder mass = "0.1" length = "0.026" radius = "0.09704">
+        <xacro:inertial_cylinder mass = "0.1" length = "0.041" radius = "0.09704">
             <origin xyz = "0 0 0" rpy = "0 0 0"/>
         </xacro:inertial_cylinder>
@@ -119,5 +119,5 @@
         <parent link = "base_link"/>
         <child link = "right_wheel"/>
-        <origin xyz = "0 -0.101 0" rpy = "${pi/2} 0 0"/>
+        <origin xyz = "0 -0.110 0" rpy = "${pi/2} 0 0"/>
         <axis xyz = " 0 0 -1"/>
     </joint>
