Commit message: Added to combine 3d lidar and rover

File: description/lidar_3d.xacro (robot description, xacro)
@@ -2,5 +2,5 @@
 <robot xmlns:xacro = "http://www.ros.org/wiki/xacro">
     <!-- Lidar Link -->
-    <link name = "laser_frame">
+    <link name = "laser_3d_frame">
         <visual>
             <origin xyz = "0 0 0" rpy = "0 0 0"/>
@@ -20,9 +20,9 @@
         </xacro:inertial_cylinder>
     </link>
-    <gazebo reference = "laser_frame">
+    <gazebo reference = "laser_3d_frame">
         <material>
             Gazebo/Red
         </material>
-        <sensor name = "laser" type = "ray">
+        <sensor name = "laser_3d" type = "ray">
             <pose> 0 0 0 0 0 0 </pose>
             <visualize>false</visualize>
@@ -41,18 +41,18 @@
                 </range>
             </ray>
-            <plugin name = "laser_controller" filename = "libgazebo_ros_ray_sensor.so">
+            <plugin name = "laser_3d_controller" filename = "libgazebo_ros_ray_sensor.so">
                 <ros>
-                    <argument>~/out:=scan</argument>
+                    <argument>~/out:=scan_3d</argument>
                 </ros>
                 <output_type>sensor_msgs/LaserScan</output_type>
-                <frame_name>laser_frame</frame_name>
+                <frame_name>laser_3d_frame</frame_name>
             </plugin>
         </sensor>
     </gazebo>
     <!-- Lidar Joint -->
-    <joint name = "laser_joint" type = "fixed">
-        <parent link = "chassis"/>
-        <child link = "laser_frame"/>
-        <origin xyz = "0.125 0 0.123" rpy = "0 0 0"/>
+    <joint name = "laser_3d_joint" type = "fixed">
+        <parent link = "bracket_link"/>
+        <child link = "laser_3d_frame"/>
+        <origin xyz = "0 0 0.051" rpy = "0 ${pi/2} 0"/>
     </joint>
 </robot>

File: description/robot.urdf.xacro (robot description, xacro)
@@ -11,4 +11,5 @@
     </xacro:unless>
     <xacro:include filename = "lidar.xacro"/>
+    <xacro:include filename = "lidar_3d.xacro"/>
     <xacro:include filename = "camera.xacro"/>
     <!-- <xacro:include filename = "depth_camera.xacro"/> -->

File: description/robot_core.xacro (robot description, xacro)
@@ -60,4 +60,110 @@
         <origin xyz = "-0.125 0 0"/>
     </joint>
+    <!-- Stepper Link -->
+    <link name="stepper_link">
+        <visual>
+            <origin xyz="0 0 0.0415"/>
+            <geometry>
+                <box size="0.048 0.048 0.043"/>
+            </geometry>
+            <material name="black"/>
+        </visual>
+        <collision>
+            <origin xyz="0 0 0.0415"/>
+            <geometry>
+                <box size="0.048 0.048 0.043"/>
+            </geometry>
+        </collision>
+        <xacro:inertial_box mass = "0.5" x = "0.048" y = "0.048" z = "0.043">
+            <origin xyz = "0 0 0.0415" rpy = "0 0 0"/>
+        </xacro:inertial_box>
+    </link>
+    <gazebo reference="stepper_link">
+        <material>
+            Gazebo/Black
+        </material>
+    </gazebo>
+    <!-- Stepper Joint -->
+    <joint name="stepper_joint" type="fixed">
+        <parent link="base_link"/>
+        <child link="stepper_link"/>
+        <origin xyz="0 0 0.123"/>
+    </joint>
+    <!-- Shaft Link -->
+    <link name="shaft_link">
+        <visual>
+            <origin xyz="0 0 0.018"/>
+            <geometry>
+                <cylinder radius="0.01" length="0.036"/>
+            </geometry>
+            <material name="orange"/>
+        </visual>
+        <collision>
+            <origin xyz="0 0 0.018"/>
+            <geometry>
+                <cylinder radius="0.01" length="0.036"/>
+            </geometry>
+        </collision>
+        <xacro:inertial_cylinder mass = "0.1" length = "0.036" radius = "0.01">
+            <origin xyz = "0 0 0.018" rpy = "0 0 0"/>
+        </xacro:inertial_cylinder>
+    </link>
+    <gazebo reference="shaft_link">
+        <material>
+            Gazebo/Orange
+        </material>
+    </gazebo>
+    <!-- Shaft Joint -->
+    <joint name="shaft_joint" type="fixed">
+        <parent link="stepper_link"/>
+        <child link="shaft_link"/>
+        <origin xyz="0 0 0.043" rpy="0 0 0"/>
+    </joint>
+    <!-- Bracket Link -->
+    <link name="bracket_link">
+        <visual>
+            <origin xyz="-0.012 0 0.005"/>
+            <geometry>
+                <box size="0.045 0.03 0.01"/>
+            </geometry>
+            <material name="white"/>
+        </visual>
+        <collision>
+            <origin xyz="-0.012 0 0.005"/>
+            <geometry>
+                <box size="0.045 0.03 0.01"/>
+            </geometry>
+        </collision>
+        <xacro:inertial_box mass = "0.1" x = "0.045" y = "0.03" z = "0.01">
+            <origin xyz = "0 -0.012 0.005" rpy = "0 0 0"/>
+        </xacro:inertial_box>
+        <visual>
+            <origin xyz="-0.0255 0 0.050" rpy="0 ${pi/2} 0"/>
+            <geometry>
+                <cylinder radius="0.0415" length="0.018"/>
+            </geometry>
+            <material name="white"/>
+        </visual>
+        <collision>
+            <origin xyz="-0.0255 0 0.050" rpy="0 ${pi/2} 0"/>
+            <geometry>
+                <cylinder radius="0.0415" length="0.018"/>
+            </geometry>
+        </collision>
+        <xacro:inertial_cylinder mass = "0.1" length = "0.018" radius = "0.0415">
+            <origin xyz = "-0.0255 0 0.050" rpy="0 ${pi/2} 0"/>
+        </xacro:inertial_cylinder>
+    </link>
+    <gazebo reference="bracket_link">
+        <material>
+            Gazebo/White
+        </material>
+    </gazebo>
+    <!-- Bracket Joint -->
+    <joint name="bracket_joint" type="fixed">
+        <parent link="shaft_link"/>
+        <child link="bracket_link"/>
+        <origin xyz="0 0 0.036" rpy="0 0 0"/>
+    </joint>
     <!-- Left Wheel Link -->
     <link name = "left_wheel">
